File: kicad-pmod-ext.kicad_pcb (KiCad board)
At the start: 2 copper layers, 0 parts

Commit message: 1.0
Parts:
- added D1: green, LED_SMD:LED_0603_1608Metric_Pad1.05x0.95mm_HandSolder, F.Cu at (120.7, 81.3)
- added H1: 2.5, MountingHole:MountingHole_2.5mm, F.Cu at (120.7, 95.2)
- added J1: pmod-4, Library:PinHeader_2x06_P2.54mm_Horizontal, F.Cu at (127.0, 76.2)
- added J2: pmod-4 cable, Connector_PinSocket_2.54mm:PinSocket_2x06_P2.54mm_Vertical, F.Cu at (127.0, 90.2)
- added R1: 4k7, Resistor_SMD:R_0603_1608Metric_Pad0.98x0.95mm_HandSolder, F.Cu at (115.2, 81.3)
Routing:
- net +3.3V: track 0.00 -> 22.9 mm
- net /pmod8: track 0.00 -> 17.6 mm
- net /pmod4: track 0.00 -> 17.6 mm
- net /pmod2: track 0.00 -> 17.6 mm
- net /pmod6: track 0.00 -> 17.5 mm
- net GND: track 0.00 -> 16.5 mm
- net /pmod7: track 0.00 -> 11.4 mm
- net /pmod5: track 0.00 -> 11.4 mm
- net /pmod3: track 0.00 -> 11.4 mm
- net /pmod1: track 0.00 -> 11.4 mm
- net Net-(D1-A): track 0.00 -> 3.65 mm
- added copper zone on B.Cu, net GND
- added copper zone on F.Cu, net GND
Other:
- board outline added: 16.5 x 27.9 mm
- board text added: "+3V3"
- board text added: "PMOD Extension by S59MZ"
- board text added: "gnd"

Commit message: 1.0
Connections:
- J2 pad 1: /pmod2 -> /pmod1
- J2 pad 2: /pmod1 -> /pmod2
- J2 pad 3: /pmod4 -> /pmod3
- J2 pad 4: /pmod3 -> /pmod4
- J2 pad 5: /pmod6 -> /pmod5
- J2 pad 6: /pmod5 -> /pmod6
- J2 pad 7: /pmod8 -> /pmod7
- J2 pad 8: /pmod7 -> /pmod8
Routing:
- net /pmod7: track 11.4 -> 15.0 mm
- net /pmod5: track 11.4 -> 15.0 mm
- net /pmod3: track 11.4 -> 15.0 mm
- net /pmod1: track 11.4 -> 15.0 mm
- net /pmod8: track 17.6 -> 15.0 mm
- net /pmod4: track 17.6 -> 15.0 mm
- net /pmod2: track 17.6 -> 15.0 mm
- net /pmod6: track 17.5 -> 15.0 mm
Changed lines of the file:
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@@
       (stroke (width 0.1) (type solid)) (layer "F.Fab"))
     (pad "1" thru_hole rect (at 0 0 270) (size 1.7 1.7) (drill 1) (layers "*.Cu" "*.Mask")
-      (net 4 "/pmod2") (pinfunction "Pin_1") (pintype "passive"))
+      (net 3 "/pmod1") (pinfunction "Pin_1") (pintype "passive"))
     (pad "2" thru_hole oval (at -2.54 0 270) (size 1.7 1.7) (drill 1) (layers "*.Cu" "*.Mask")
-      (net 3 "/pmod1") (pinfunction "Pin_2") (pintype "passive"))
+      (net 4 "/pmod2") (pinfunction "Pin_2") (pintype "passive"))
     (pad "3" thru_hole oval (at 0 2.54 270) (size 1.7 1.7) (drill 1) (layers "*.Cu" "*.Mask")
-      (net 6 "/pmod4") (pinfunction "Pin_3") (pintype "passive"))
+      (net 5 "/pmod3") (pinfunction "Pin_3") (pintype "passive"))
     (pad "4" thru_hole oval (at -2.54 2.54 270) (size 1.7 1.7) (drill 1) (layers "*.Cu" "*.Mask")
-      (net 5 "/pmod3") (pinfunction "Pin_4") (pintype "passive"))
+      (net 6 "/pmod4") (pinfunction "Pin_4") (pintype "passive"))
     (pad "5" thru_hole oval (at 0 5.08 270) (size 1.7 1.7) (drill 1) (layers "*.Cu" "*.Mask")
-      (net 8 "/pmod6") (pinfunction "Pin_5") (pintype "passive"))
+      (net 7 "/pmod5") (pinfunction "Pin_5") (pintype "passive"))
     (pad "6" thru_hole oval (at -2.54 5.08 270) (size 1.7 1.7) (drill 1) (layers "*.Cu" "*.Mask")
-      (net 7 "/pmod5") (pinfunction "Pin_6") (pintype "passive"))
+      (net 8 "/pmod6") (pinfunction "Pin_6") (pintype "passive"))
     (pad "7" thru_hole oval (at 0 7.62 270) (size 1.7 1.7) (drill 1) (layers "*.Cu" "*.Mask")
-      (net 10 "/pmod8") (pinfunction "Pin_7") (pintype "passive"))
+      (net 9 "/pmod7") (pinfunction "Pin_7") (pintype "passive"))
     (pad "8" thru_hole oval (at -2.54 7.62 270) (size 1.7 1.7) (drill 1) (layers "*.Cu" "*.Mask")
-      (net 9 "/pmod7") (pinfunction "Pin_8") (pintype "passive"))
+      (net 10 "/pmod8") (pinfunction "Pin_8") (pintype "passive"))
     (pad "9" thru_hole oval (at 0 10.16 270) (size 1.7 1.7) (drill 1) (layers "*.Cu" "*.Mask")
       (net 1 "GND") (pinfunction "Pin_9") (pintype "passive"))
@@
   (segment (start 116.84 90.17) (end 116.84 73.66) (width 0.75) (layer "B.Cu") (net 1))
   (segment (start 119.775 81.28) (end 116.125 81.28) (width 0.25) (layer "F.Cu") (net 2))
-  (segment (start 127 76.2) (end 127 87.63) (width 0.25) (layer "B.Cu") (net 3))
-  (segment (start 127 73.66) (end 125.73 74.93) (width 0.25) (layer "B.Cu") (net 4))
-  (segment (start 125.73 88.9) (end 127 90.17) (width 0.25) (layer "B.Cu") (net 4))
-  (segment (start 125.73 74.93) (end 125.73 88.9) (width 0.25) (layer "B.Cu") (net 4))
-  (segment (start 124.46 87.63) (end 124.46 76.2) (width 0.25) (layer "B.Cu") (net 5))
-  (segment (start 123.19 88.9) (end 124.46 90.17) (width 0.25) (layer "B.Cu") (net 6))
-  (segment (start 123.19 74.93) (end 123.19 88.9) (width 0.25) (layer "B.Cu") (net 6))
-  (segment (start 124.46 73.66) (end 123.19 74.93) (width 0.25) (layer "B.Cu") (net 6))
-  (segment (start 121.92 87.63) (end 121.92 76.2) (width 0.25) (layer "B.Cu") (net 7))
-  (segment (start 120.745 74.835) (end 120.745 88.995) (width 0.25) (layer "B.Cu") (net 8))
-  (segment (start 120.745 88.995) (end 121.92 90.17) (width 0.25) (layer "B.Cu") (net 8))
-  (segment (start 121.92 73.66) (end 120.745 74.835) (width 0.25) (layer "B.Cu") (net 8))
-  (segment (start 119.38 87.63) (end 119.38 76.2) (width 0.25) (layer "B.Cu") (net 9))
-  (segment (start 118.11 88.9) (end 119.38 90.17) (width 0.25) (layer "B.Cu") (net 10))
-  (segment (start 119.38 73.66) (end 118.11 74.93) (width 0.25) (layer "B.Cu") (net 10))
-  (segment (start 118.11 74.93) (end 118.11 88.9) (width 0.25) (layer "B.Cu") (net 10))
+  (segment (start 127 79.375) (end 127 76.2) (width 0.25) (layer "B.Cu") (net 3))
+  (segment (start 125.73 88.9) (end 127 90.17) (width 0.25) (layer "B.Cu") (net 3))
+  (segment (start 125.73 80.645) (end 127 79.375) (width 0.25) (layer "B.Cu") (net 3))
+  (segment (start 125.73 88.9) (end 125.73 80.645) (width 0.25) (layer "B.Cu") (net 3))
+  (segment (start 128.27 79.375) (end 128.27 74.93) (width 0.25) (layer "B.Cu") (net 4))
+  (segment (start 127 87.63) (end 127 80.645) (width 0.25) (layer "B.Cu") (net 4))
+  (segment (start 127 80.645) (end 128.27 79.375) (width 0.25) (layer "B.Cu") (net 4))
+  (segment (start 128.27 74.93) (end 127 73.66) (width 0.25) (layer "B.Cu") (net 4))
+  (segment (start 124.46 79.375) (end 124.46 76.2) (width 0.25) (layer "B.Cu") (net 5))
+  (segment (start 123.19 80.645) (end 124.46 79.375) (width 0.25) (layer "B.Cu") (net 5))
+  (segment (start 123.19 88.9) (end 123.19 80.645) (width 0.25) (layer "B.Cu") (net 5))
+  (segment (start 123.19 88.9) (end 124.46 90.17) (width 0.25) (layer "B.Cu") (net 5))
+  (segment (start 124.46 80.645) (end 124.46 87.63) (width 0.25) (layer "B.Cu") (net 6))
+  (segment (start 125.73 79.375) (end 124.46 80.645) (width 0.25) (layer "B.Cu") (net 6))
+  (segment (start 124.46 73.66) (end 125.73 74.93) (width 0.25) (layer "B.Cu") (net 6))
+  (segment (start 125.73 74.93) (end 125.73 79.375) (width 0.25) (layer "B.Cu") (net 6))
+  (segment (start 120.65 80.645) (end 121.92 79.375) (width 0.25) (layer "B.Cu") (net 7))
+  (segment (start 121.92 79.375) (end 121.92 76.2) (width 0.25) (layer "B.Cu") (net 7))
+  (segment (start 120.65 88.9) (end 120.65 80.645) (width 0.25) (layer "B.Cu") (net 7))
+  (segment (start 121.92 90.17) (end 120.65 88.9) (width 0.25) (layer "B.Cu") (net 7))
+  (segment (start 123.19 79.375) (end 121.92 80.645) (width 0.25) (layer "B.Cu") (net 8))
+  (segment (start 121.92 73.66) (end 123.19 74.93) (width 0.25) (layer "B.Cu") (net 8))
+  (segment (start 121.92 80.645) (end 121.92 87.63) (width 0.25) (layer "B.Cu") (net 8))
+  (segment (start 123.19 74.93) (end 123.19 79.375) (width 0.25) (layer "B.Cu") (net 8))
+  (segment (start 118.11 88.9) (end 119.38 90.17) (width 0.25) (layer "B.Cu") (net 9))
+  (segment (start 119.38 79.375) (end 119.38 76.2) (width 0.25) (layer "B.Cu") (net 9))
+  (segment (start 118.11 80.645) (end 119.38 79.375) (width 0.25) (layer "B.Cu") (net 9))
+  (segment (start 118.11 88.9) (end 118.11 80.645) (width 0.25) (layer "B.Cu") (net 9))
+  (segment (start 119.38 73.66) (end 120.65 74.93) (width 0.25) (layer "B.Cu") (net 10))
+  (segment (start 120.65 74.93) (end 120.65 79.375) (width 0.25) (layer "B.Cu") (net 10))
+  (segment (start 120.65 79.375) (end 119.38 80.645) (width 0.25) (layer "B.Cu") (net 10))
+  (segment (start 119.38 80.645) (end 119.38 87.63) (width 0.25) (layer "B.Cu") (net 10))
   (segment (start 114.3 81.28) (end 114.3 87.63) (width 0.75) (layer "F.Cu") (net 11))
   (segment (start 114.3 73.66) (end 114.3 90.17) (width 0.75) (layer "B.Cu") (net 11))
