File: kicad-pmod-ext.kicad_sch (KiCad schematic)
At the start: 0 parts

Commit message: 1.0
Parts:
- added D1: green, LED_SMD:LED_0603_1608Metric_Pad1.05x0.95mm_HandSolder, symbol Device:LED
- added H1: 2.5, MountingHole:MountingHole_2.5mm, symbol Mechanical:MountingHole
- added J1: pmod-4, Library:PinHeader_2x06_P2.54mm_Horizontal, symbol Connector_Generic:Conn_02x06_Odd_Even
- added J2: pmod-4 cable, Connector_PinSocket_2.54mm:PinSocket_2x06_P2.54mm_Vertical, symbol Connector_Generic:Conn_02x06_Odd_Even
- added R1: 4k7, Resistor_SMD:R_0603_1608Metric_Pad0.98x0.95mm_HandSolder, symbol Device:R
Connections:
- new net: D1.2 (A), R1.2
- new net +3.3V: J1.11 (Pin_11), J1.12 (Pin_12), J2.11 (Pin_11), J2.12 (Pin_12), R1.1
- new net GND: D1.1 (K), J1.10 (Pin_10), J1.9 (Pin_9), J2.10 (Pin_10), J2.9 (Pin_9)
- new net pmod1: J1.1 (Pin_1), J2.2 (Pin_2)
- new net pmod2: J1.2 (Pin_2), J2.1 (Pin_1)
- new net pmod3: J1.3 (Pin_3), J2.4 (Pin_4)
- new net pmod4: J1.4 (Pin_4), J2.3 (Pin_3)
- new net pmod5: J1.5 (Pin_5), J2.6 (Pin_6)
- new net pmod6: J1.6 (Pin_6), J2.5 (Pin_5)
- new net pmod7: J1.7 (Pin_7), J2.8 (Pin_8)
- new net pmod8: J1.8 (Pin_8), J2.7 (Pin_7)

Commit message: 1.0
Connections:
- net pmod1: now also J2.1 (Pin_1); no longer J2.2 (Pin_2)
- net pmod2: now also J2.2 (Pin_2); no longer J2.1 (Pin_1)
- net pmod3: now also J2.3 (Pin_3); no longer J2.4 (Pin_4)
- net pmod4: now also J2.4 (Pin_4); no longer J2.3 (Pin_3)
- net pmod5: now also J2.5 (Pin_5); no longer J2.6 (Pin_6)
- net pmod6: now also J2.6 (Pin_6); no longer J2.5 (Pin_5)
- net pmod7: now also J2.7 (Pin_7); no longer J2.8 (Pin_8)
- net pmod8: now also J2.8 (Pin_8); no longer J2.7 (Pin_7)
Changed lines of the file:
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@@
     (stroke (width 0) (type default))
+  )
+  (label "pmod2" (at 119.38 99.06 180) (fields_autoplaced)
+    (effects (font (size 1.27 1.27)) (justify right bottom))
+  )
+  (label "pmod6" (at 119.38 104.14 180) (fields_autoplaced)
+    (effects (font (size 1.27 1.27)) (justify right bottom))
+  )
+  (label "pmod8" (at 119.38 106.68 180) (fields_autoplaced)
+    (effects (font (size 1.27 1.27)) (justify right bottom))
   )
   (label "pmod2" (at 119.38 66.04 180) (fields_autoplaced)
     (effects (font (size 1.27 1.27)) (justify right bottom))
-  )
-  (label "pmod8" (at 132.08 106.68 0) (fields_autoplaced)
-    (effects (font (size 1.27 1.27)) (justify left bottom))
   )
   (label "pmod5" (at 132.08 71.12 0) (fields_autoplaced)
@@
     (effects (font (size 1.27 1.27)) (justify left bottom))
   )
+  (label "pmod7" (at 132.08 106.68 0) (fields_autoplaced)
+    (effects (font (size 1.27 1.27)) (justify left bottom))
+  )
   (label "pmod1" (at 132.08 66.04 0) (fields_autoplaced)
     (effects (font (size 1.27 1.27)) (justify left bottom))
   )
-  (label "pmod2" (at 132.08 99.06 0) (fields_autoplaced)
+  (label "pmod3" (at 132.08 101.6 0) (fields_autoplaced)
     (effects (font (size 1.27 1.27)) (justify left bottom))
   )
@@
     (effects (font (size 1.27 1.27)) (justify right bottom))
   )
+  (label "pmod5" (at 132.08 104.14 0) (fields_autoplaced)
+    (effects (font (size 1.27 1.27)) (justify left bottom))
+  )
   (label "pmod8" (at 119.38 73.66 180) (fields_autoplaced)
-    (effects (font (size 1.27 1.27)) (justify right bottom))
-  )
-  (label "pmod5" (at 119.38 104.14 180) (fields_autoplaced)
     (effects (font (size 1.27 1.27)) (justify right bottom))
   )
@@
     (effects (font (size 1.27 1.27)) (justify right bottom))
   )
-  (label "pmod6" (at 132.08 104.14 0) (fields_autoplaced)
-    (effects (font (size 1.27 1.27)) (justify left bottom))
+  (label "pmod4" (at 119.38 101.6 180) (fields_autoplaced)
+    (effects (font (size 1.27 1.27)) (justify right bottom))
   )
   (label "pmod3" (at 132.08 68.58 0) (fields_autoplaced)
     (effects (font (size 1.27 1.27)) (justify left bottom))
   )
-  (label "pmod4" (at 132.08 101.6 0) (fields_autoplaced)
+  (label "pmod1" (at 132.08 99.06 0) (fields_autoplaced)
     (effects (font (size 1.27 1.27)) (justify left bottom))
   )
-  (label "pmod7" (at 119.38 106.68 180) (fields_autoplaced)
-    (effects (font (size 1.27 1.27)) (justify right bottom))
-  )
-  (label "pmod3" (at 119.38 101.6 180) (fields_autoplaced)
-    (effects (font (size 1.27 1.27)) (justify right bottom))
-  )
-  (label "pmod1" (at 119.38 99.06 180) (fields_autoplaced)
-    (effects (font (size 1.27 1.27)) (justify right bottom))
-  )
   (symbol (lib_id "power:GND") (at 119.38 109.22 270) (unit 1)
